File: solar_mains_charge_manager/solar_mains_charge_manager.brd (EAGLE design)
At the start: 100 x 80 mm, 8 parts, among them X10 22-23-2041, X2 22-23-2021, X3 22-23-2031, X5 22-23-2031, X6 22-23-2041, X7 53047-15, X8 53047-15

Commit message: Stuff
Parts:
- removed X10, X6: 22-23-2041, con-molex:22-23-2041
- removed X3, X5: 22-23-2031, con-molex:22-23-2031
- removed X7, X8: 53047-15, con-molex:53047-15
- added C1, C2, C6: (no value), capacitor-wima:C2.5-3
- added D1: (no value), diode:DO34Z7
- added F-1: (no value), qfm-trx1-24g:FUSE
- added JMP1, JMP2, JMP3: 0R-JUMPA, jump-0r-smd:A0R-JMP
- added R1, R11, R12, R13, R14, R15, R16, R17: (no value), rcl:0204/5
- added R10, R2, R3, R4, R5, R6, R7, R8, R9: (no value), resistor:0204V
- added R19: (no value), resistor:0204/5
- added S1, S2, S3: (no value), switch-omron:B3F-10XX
- added SJ1, SJ10, SJ11, SJ12: (no value), jumper:SJ
- added SV1, SV2: (no value), con-lsta:FE15
- added SV3, SV8: (no value), con-lstb:MA04-1
- added SV4, SV5, SV6, SV7: (no value), con-lstb:MA07-1
- added SV9: (no value), con-lstb:MA03-1
- added TIP122: IRF530, transistor-power:TO220BV
- added V-REG-1: (no value), qfm-trx1-24g:TO92
- added X1: 22-23-2021, con-molex:22-23-2021
- U$1: device Arduino-clone:NANO -> nano_without_those_headers:NANO
- moved X2 25.5 mm to (28.3, 76.7), turned to 0 degrees
- moved U$1 25.4 mm to (24.5, 25.4)
Connections:
- removed net 12V: U$1.RAW, X5.3, X7.1
- removed net 12V1: U$1.AREF, X2.1, X7.13
- removed net N$17: U$1.D11, X3.2, X8.2
- removed net N$19: U$1.D9, X6.3, X8.4
- removed net N$22: U$1.D7, X8.6
- removed net N$23: U$1.D6, X8.7
- removed net N$27: U$1.D2, X8.11
- removed net N$28: U$1.GND1, X8.12
- removed net N$32: U$1.5V, X7.4
- removed net N$33: U$1.A7, X7.5
- removed net N$34: U$1.A6, X7.6
- removed net N$35: U$1.A5, X7.7
- removed net N$36: U$1.A4, X7.8
- removed net N$37: U$1.A3, X7.9
- removed net N$38: U$1.A2, X7.10
- removed net N$39: U$1.A1, X7.11
- removed net N$40: U$1.A0, X7.12
- removed net N$41: X10.4
- removed net N$42: X10.3
- new net 5V: SJ1.1, SJ12.2, SV1.4, SV3.3, SV6.1, SV6.2, SV6.3, SV6.4, SV6.5, SV6.6, SV6.7, SV8.3, SV9.3, U$1.5V
- new net A0: R1.2, R8.1, U$1.A0
- new net A1: R11.2, R7.1, U$1.A1
- new net A2: R12.2, R6.1, U$1.A2
- new net A3: R13.2, R5.1, U$1.A3
- new net A4: JMP3.1, R14.2, R4.1, U$1.A4
- new net A5: JMP2.1, R15.2, R3.1, U$1.A5
- new net A6: R10.1, R16.2, U$1.A6
- new net A7: R17.2, R9.1, SV9.1, U$1.A7
- new net AREF: SJ1.2, SV1.13, U$1.AREF
- new net D8: S2.1, SV2.5, U$1.D8
- new net D9: S1.2, SV2.4, U$1.D9
- new net N$1: C1.1, R19.2, SJ11.1, TIP122.S
- new net N$13: JMP3.2, SV3.1
- new net N$3: C6.1, D1.C, R19.1, R2.2, TIP122.G
- new net N$4: SV2.1, U$1.D12
- new net N$6: JMP1.3, V-REG-1.2
- new net N$7: SV2.2, U$1.D11
- new net N$8: F-1.P$1, X2.2
- new net RELAY: SV2.7, U$1.D6, X1.2
- new net RST: S3.2, SV1.3, U$1.RST
- new net SCLSW: JMP2.3, SV2.11, U$1.D2
- new net SDASW: JMP3.3, SV2.6, U$1.D7
- new net VD0: R8.2, SJ10.2, SV1.12
- new net VD1: R7.2, SV1.11
- new net VD2: R6.2, SV1.10
- new net VD3: R5.2, SV1.9
- new net VD4: R4.2, SV1.8
- new net VD5: R3.2, SV1.7
- new net VD6: R10.2, SV1.6
- new net VD7: R9.2, SV1.5
- new net VIN: JMP1.1, SV1.1, U$1.RAW
- net BAT: now also F-1.P$2, R2.1, SJ10.1, SV4.1, SV4.2, SV4.3, SV4.4, SV4.5, SV4.6, SV4.7, SV8.1, TIP122.D; no longer X10.2, X5.2
- net GND: now also C1.2, C2.2, C6.2, D1.A, R1.1, R11.1, R12.1, R13.1, R14.1, R15.1, R16.1, R17.1, S1.4, S2.4, S3.4, SV1.2, SV2.12, SV3.4, SV7.1, SV7.2, SV7.3, SV7.4, SV7.5, SV7.6, SV7.7, SV8.4, SV9.2, U$1.GND1, V-REG-1.1, X1.1, X2.1; no longer X10.1, X3.1, X5.1, X6.1, X7.2
- net N$12: now also JMP2.2, SV3.2; no longer U$1.D12, X8.1
- net N$18: now also SV2.3; no longer X3.3, X8.3
- net N$2: now also SV1.15; no longer X7.15
- net N$20: now also C2.1, SJ12.1, V-REG-1.3; no longer U$1.D8, X6.4, X8.5
- net N$21: now also JMP1.2, SJ11.2, SV5.1, SV5.2, SV5.3, SV5.4, SV5.5, SV5.6, SV5.7, SV8.2; no longer U$1.RST, X6.2, X7.3
- net N$24: now also SV2.8; no longer X8.8
- net N$25: now also SV2.9; no longer X8.9
- net N$26: now also SV2.10; no longer X8.10
- net N$29: now also SV2.13; no longer X8.13
- net N$30: now also SV2.14; no longer X8.14
- net N$31: now also SV2.15; no longer X8.15
- net N$5: now also SV1.14; no longer X2.2, X7.14
Routing:
- net VIN: track 0.00 -> 126.8 mm
- net 5V: track 0.00 -> 119.5 mm
- net D9: track 0.00 -> 57.4 mm
- net D8: track 0.00 -> 56.8 mm
- net BAT: track 0.00 -> 45.1 mm
- net N$21: track 0.00 -> 38.8 mm
- net VD0: track 0.00 -> 35.5 mm
- net RELAY: track 0.00 -> 28.8 mm
- net SCLSW: track 0.00 -> 27.5 mm
- net A4: track 0.00 -> 27.1 mm
- net RST: track 0.00 -> 25.1 mm
- net A5: track 0.00 -> 23.4 mm
- net N$3: track 0.00 -> 17.0 mm
- net SDASW: track 0.00 -> 16.1 mm
- net AREF: track 0.00 -> 14.8 mm
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- added copper zone on layer 1, net GND
- added copper zone on layer 16, net GND
Other:
- board size 100 x 80 mm -> 42 x 80 mm
- board text added: "12V"
- board text added: "5V"
- board text added: "BAT"
- board text added: "Display"
- board text added: "GND"
- board text added: "RST"
- board text added: "Relay"
